File: analoge.kicad_sch (KiCad schematic)
At the start: 32 parts, among them U10 LT1097S8, U5 AD8656, U6 REF3450T, U7 IM68A130A, U8 MCP33131, U9 LP5907MFX-2.5

Commit message: Leitete und beendete am meisten die Leiterplatte.
Parts:
- C34: value 7.5n -> 6.8n
- C36: value 7.5n -> 3n
- R16: value 13.8k -> 16k
Changed lines of the file:
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@@
 		)
 	)
-	(text_box "Des ADUs Datenblatt sagt, dass der Kondensator des VREFs tantal sein soll."
+	(text_box "Das Datenblatt des ADUs sagt, dass der Kondensator des VREFs tantal sein soll."
 		(exclude_from_sim no)
 		(at 208.28 36.83 0)
@@
 		)
 	)
+	(text_box "15.9 mVpp bei 90 dB(SPL), 1 kHz"
+		(exclude_from_sim no)
+		(at 69.85 50.8 0)
+		(size 25.4 6.35)
+		(stroke
+			(width 0)
+			(type default)
+		)
+		(fill
+			(type none)
+		)
+		(effects
+			(font
+				(size 1.27 1.27)
+			)
+			(justify left top)
+		)
+	)
+	(text_box "Die Verstärkung sei um 44 dB."
+		(exclude_from_sim no)
+		(at 63.5 88.9 0)
+		(size 19.05 6.35)
+		(stroke
+			(width 0)
+			(type default)
+		)
+		(fill
+			(type none)
+		)
+		(effects
+			(font
+				(size 1.27 1.27)
+			)
+			(justify left top)
+		)
+	)
+	(text_box "In LTspice war die Bandbreite um 24 kHz bei -3 dB und um 180 kHz bei -40 dB."
+		(exclude_from_sim no)
+		(at 139.7 88.9 0)
+		(size 25.4 12.7)
+		(stroke
+			(width 0)
+			(type default)
+		)
+		(fill
+			(type none)
+		)
+		(effects
+			(font
+				(size 1.27 1.27)
+			)
+			(justify left top)
+		)
+	)
 	(text_box "Beide Kondensator an der Referenz müssen niederen ESW haben."
 		(exclude_from_sim no)
@@
 		)
 	)
+	(text_box "2.5 Vpp bei 90 dB(SPL), 1 kHz"
+		(exclude_from_sim no)
+		(at 107.95 88.9 0)
+		(size 25.4 6.35)
+		(stroke
+			(width 0)
+			(type default)
+		)
+		(fill
+			(type none)
+		)
+		(effects
+			(font
+				(size 1.27 1.27)
+			)
+			(justify left top)
+		)
+	)
 	(text_box "Der ESW darf höchstens 500 mΩ sein."
 		(exclude_from_sim no)
@@
 			)
 		)
-		(property "Value" "7.5n"
+		(property "Value" "3n"
 			(at 137.16 76.1999 0)
 			(effects
@@
 			)
 		)
-		(property "Value" "7.5n"
+		(property "Value" "6.8n"
 			(at 140.97 57.15 90)
 			(effects
@@
 			)
 		)
-		(property "Value" "13.8k"
+		(property "Value" "16k"
 			(at 101.6 78.74 90)
 			(effects
