File: hsa_r0.kicad_pcb (KiCad board)
At the start: 2 copper layers, 77.5 x 50 mm, 103 parts, among them J1 USB_B_Micro, J2 Conn_02x05_Odd_Even, J3 Conn_01x12_Socket, J4 Conn_01x02_Pin, Q1 2N7002, Q2 2N7002, SW1 SW_Omron_B3FS, SW10 RotaryEncoder, SW11 RotaryEncoder, SW2 SW_Omron_B3FS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

Commit message: Leitete und beendete am meisten die Leiterplatte.
Parts:
- added REF**: MountingHole_3.2mm_M3_ISO7380_Pad_TopBottom, MountingHole:MountingHole_3.2mm_M3_ISO7380_Pad_TopBottom, F.Cu at (135.0, 85.0)
- C34: value 7.5n -> 6.8n
- C36: value 7.5n -> 3n
- J4: moved to F.Cu
- moved Q2 33.1 mm to (191.8, 81.9)
- moved D1 33.1 mm to (191.8, 85.0), turned to 180 degrees
- moved R11 31.5 mm to (191.8, 86.8), turned to 0 degrees
- moved C38 25.8 mm to (135.0, 52.5), turned to 180 degrees
- moved U9 19.2 mm to (135.0, 55.8), turned to -90 degrees
- moved J4 17.8 mm to (174.8, 52.5), turned to 0 degrees
- moved C39 12.8 mm to (135.0, 59.0), turned to 180 degrees
- moved C26 9.53 mm to (153.2, 57.5), turned to -90 degrees
- moved R2 8.02 mm to (186.5, 79.5), turned to 0 degrees
- moved C11 6.91 mm to (165.0, 43.8), turned to 180 degrees
- moved R8 6.91 mm to (165.0, 45.2), turned to 180 degrees
- moved C22 6.91 mm to (178.0, 50.7), turned to 90 degrees
- moved C23 6.21 mm to (182.5, 46.0), turned to 180 degrees
- moved C33 4.74 mm to (137.5, 63.2), turned to 180 degrees
- moved U4 4.51 mm to (147.5, 56.2), turned to 180 degrees
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Connections:
- C23 pad 1: +3.3V -> +3V3
- U1 pad 37: unconnected-(U1-PE7-Pad37) -> /Prozessor/SW_0
- U1 pad 38: unconnected-(U1-PE8-Pad38) -> /Prozessor/SW_1
- U1 pad 39: unconnected-(U1-PE9-Pad39) -> /Prozessor/SW_2
- U1 pad 40: unconnected-(U1-PE10-Pad40) -> /Prozessor/SW_3
- U1 pad 41: unconnected-(U1-PE11-Pad41) -> /Prozessor/SW_4
- U1 pad 42: unconnected-(U1-PE12-Pad42) -> /Prozessor/SW_5
- U2 pad 2: +3.3V -> +3V3
Routing:
- net GNDA: track 0.00 -> 99.6 mm, vias 0 -> 123
- net +3V3: track 0.00 -> 64.8 mm, vias 0 -> 21
- net /Prozessor/SW_5: track 0.00 -> 47.8 mm, vias 0 -> 1
- net /Prozessor/DK1_A: track 0.00 -> 46.4 mm, vias 0 -> 1
- net /Prozessor/DK1_B: track 0.00 -> 41.5 mm, vias 0 -> 1
- net /Prozessor/SW_4: track 0.00 -> 38.1 mm, vias 0 -> 1
- net /Prozessor/DK0_A: track 0.00 -> 33.7 mm, vias 0 -> 1
- net GNDREF: track 0.00 -> 32.5 mm, vias 0 -> 2
- net /Prozessor/SW_0: track 0.00 -> 32.0 mm, vias 0 -> 1
- net /Prozessor/USB_OTG_HS_DP: track 0.00 -> 32.0 mm, vias 0 -> 2
- net /Prozessor/DK0_B: track 0.00 -> 31.6 mm, vias 0 -> 1
- net /Prozessor/USB_OTG_HS_DM: track 0.00 -> 30.9 mm, vias 0 -> 2
- net +5V: track 0.00 -> 29.9 mm, vias 0 -> 13
- net /Prozessor/LED_0: track 0.00 -> 29.4 mm, vias 0 -> 4
- net +1V8: track 0.00 -> 29.2 mm, vias 0 -> 2
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- added copper zone on F.Cu, net +3V3
- added copper zone on In2.Cu, net +3V3
- added copper zone on F.Cu, net +5V
- added copper zone on In2.Cu, net +5V
- added copper zone on B.Cu, net GNDA
- added copper zone on F.Cu, net GNDA
- added copper zone on In1.Cu, net GNDA
- added copper zone on In2.Cu, net GNDA
- added copper zone on F.Cu, net Net-(J1-Shield)
- added copper zone on F.Cu, net VBUS
- added copper zone on In2.Cu, net VBUS
Other:
- board size 77.5 x 50 mm -> 77.5 x 47.5 mm
- copper layers 2 -> 4
- board text added: "+ -"
- board text added: "240 x 320"
- board text added: "Boot"
- board text added: "C. Carlon, 2024 https://github.com /Claegtun"
- board text added: "Error 404 Nicht gefunden!"
- board text added: "Filter +44 dB: Ton -3 dB: 24 kHz -40 dB: 180 kHz"
- board text added: "GS, 5 ~ 7 V, 500 mA"
- board text added: "Handspektrum -analysator, r0"
- board text added: "Handspektrumanalysator, r0"
- board text added: "Mikrofon > Empf. -38 dB SNR. 68 dB 10 Hz - 17 kHz"
- board text added: "Reset"
- board text added: "STM32H723VxT 480 MHz"
- board text added: "SWD"
- board text added: "Ton"
- board text added: "UHF"
- board text added: "Voll. 90 dB Rausch. 26 dB"
- board text added: "[1.8 V]"
- board text added: "[2.5 V]"
- board text added: "[3.3 V]"
- board text added: "[5 V]"
