File: prozessor.kicad_sch (KiCad schematic)
At the start: 46 parts, among them J1 USB_B_Micro, J2 Conn_02x05_Odd_Even, J3 Conn_01x12_Socket, Q1 2N7002, Q2 2N7002, SW1 SW_Omron_B3FS, SW2 SW_Omron_B3FS, SW3 PTS 647 SM70 SMTR2 LFS, SW4 PTS 647 SM70 SMTR2 LFS, SW5 PTS 647 SM70 SMTR2 LFS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

Commit message: Leitete und beendete am meisten die Leiterplatte.
Connections:
- net SW_0: now also U1.37 (PE7)
- net SW_1: now also U1.38 (PE8)
- net SW_2: now also U1.39 (PE9)
- net SW_3: now also U1.40 (PE10)
- net SW_4: now also U1.41 (PE11)
- net SW_5: now also U1.42 (PE12)
- no-connect marks 64 -> 58
