File: versorgung.kicad_sch (KiCad schematic)
At the start: 11 parts, among them J4 Conn_01x02_Pin, U2 AZ1117D-ADJ, U3 NJM12856DL3-05, U4 AZ1117H-ADJ

Commit message: Leitete und beendete am meisten die Leiterplatte.
Connections:
- net +3.3V renamed +3V3
Changed lines of the file:
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@@
 			)
 		)
-		(property "Value" "+3.3V"
-			(at 102.87 76.2 90)
+		(property "Value" "+3V3"
+			(at 102.87 76.1999 90)
 			(effects
 				(font
